File: PCB/Jones.sch (KiCad schematic (older format))
At the start: 214 parts, among them J1 USB4085-GF-A_REVA, U2 ATmega32U4-MU, Y1 16MHz

Commit message: 全てのソケットにガイド線を追加。
Parts:
- SW_BS1.5u1, SW_CTL1.25u1, SW_ENT1.5u1, SW_TAB1.5u1: footprint MX_Alps_Hybrid:MXOnly-1.5U-Hotswap -> MX_Alps_Hybrid:MXOnly-1.5U-Hotswap-guide
- SW_CAPS1u1, SW_MENU/ROPT1, SW_MHEN/CMD1u1: footprint MX_Alps_Hybrid:MXOnly-1U-Hotswap -> MX_Alps_Hybrid:MXOnly-1U-Hotswap-guide
- SW_CMD1.25u1, SW_CTL1.5u1, SW_Fn1.25u1, SW_LOPT/LALT1.25u1, SW_LongCMD1.25u1, SW_LongOPT1.25, SW_RCMD/HEN1.25u1, SW_ROPT/KANA1.25u1, SW_ROPT/KANA1.25u2: footprint MX_Alps_Hybrid:MXOnly-1.25U-Hotswap -> MX_Alps_Hybrid:MXOnly-1.25U-Hotswap-guide
- SW_ENT2.25u1: footprint MX_Alps_Hybrid:MXOnly-2.25U-Hotswap-ReversedStabilizers -> MX_Alps_Hybrid:MXOnly-2.25U-Hotswap-ReversedStabilizers-guide
- SW_LSFT1.75u1, SW_RSFT1.75u1: footprint MX_Alps_Hybrid:MXOnly-1.75U-Hotswap -> MX_Alps_Hybrid:MXOnly-1.75U-Hotswap-guide
- SW_LSFT2u1, SW_LSPC2u1, SW_RSPC2u1: footprint MX_Alps_Hybrid:MXOnly-2U-Hotswap-ReversedStabilizers -> MX_Alps_Hybrid:MXOnly-2U-Hotswap-ReversedStabilizers-guide
- SW_LSPC2.25u1: footprint MX_Alps_Hybrid:MXOnly-2.25U-Hotswap -> MX_Alps_Hybrid:MXOnly-2.25U-Hotswap-guide
- SW_RSPC6.25u1: footprint MX_Alps_Hybrid:MXOnly-6.25U-Hotswap-ReversedStabilizers -> MX_Alps_Hybrid:MXOnly-6.25U-Hotswap-ReversedStabilizers-guide
Changed lines of the file:
@@
 F 0 "SW_TAB1.5u1" H 1125 3610 50  0000 C CNN
 F 1 "SW_Push" H 1125 3519 50  0000 C CNN
-F 2 "MX_Alps_Hybrid:MXOnly-1.5U-Hotswap" H 1125 3525 50  0001 C CNN
+F 2 "MX_Alps_Hybrid:MXOnly-1.5U-Hotswap-guide" H 1125 3525 50  0001 C CNN
 F 3 "~" H 1125 3525 50  0001 C CNN
 	1    1125 3325
@@
 F 0 "SW_LSFT2u1" H 1125 6110 50  0000 C CNN
 F 1 "SW_Push" H 1125 6019 50  0000 C CNN
-F 2 "MX_Alps_Hybrid:MXOnly-2U-Hotswap-ReversedStabilizers" H 1125 6025 50  0001 C CNN
+F 2 "MX_Alps_Hybrid:MXOnly-2U-Hotswap-ReversedStabilizers-guide" H 1125 6025 50  0001 C CNN
 F 3 "~" H 1125 6025 50  0001 C CNN
 	1    1125 5825
@@
 F 0 "SW_LongCMD1.25u1" H 2425 7360 50  0000 C CNN
 F 1 "SW_Push" H 2425 7269 50  0000 C CNN
-F 2 "MX_Alps_Hybrid:MXOnly-1.25U-Hotswap" H 2425 7275 50  0001 C CNN
+F 2 "MX_Alps_Hybrid:MXOnly-1.25U-Hotswap-guide" H 2425 7275 50  0001 C CNN
 F 3 "~" H 2425 7275 50  0001 C CNN
 	1    2425 7075
@@
 F 0 "SW_ENT2.25u1" H 8275 4410 50  0000 C CNN
 F 1 "SW_Push" H 8275 4319 50  0000 C CNN
-F 2 "MX_Alps_Hybrid:MXOnly-2.25U-Hotswap-ReversedStabilizers" H 8275 4325 50  0001 C CNN
+F 2 "MX_Alps_Hybrid:MXOnly-2.25U-Hotswap-ReversedStabilizers-guide" H 8275 4325 50  0001 C CNN
 F 3 "~" H 8275 4325 50  0001 C CNN
 	1    8275 4125
@@
 F 0 "SW_LOPT/LALT1.25u1" H 2425 7210 50  0000 C CNN
 F 1 "SW_Push" H 2425 7119 50  0000 C CNN
-F 2 "MX_Alps_Hybrid:MXOnly-1.25U-Hotswap" H 2425 7125 50  0001 C CNN
+F 2 "MX_Alps_Hybrid:MXOnly-1.25U-Hotswap-guide" H 2425 7125 50  0001 C CNN
 F 3 "~" H 2425 7125 50  0001 C CNN
 	1    2425 6925
@@
 F 0 "SW_Fn1.25u1" H 10225 5935 50  0000 C CNN
 F 1 "SW_Push" H 10225 5844 50  0000 C CNN
-F 2 "MX_Alps_Hybrid:MXOnly-1.25U-Hotswap" H 10225 5850 50  0001 C CNN
+F 2 "MX_Alps_Hybrid:MXOnly-1.25U-Hotswap-guide" H 10225 5850 50  0001 C CNN
 F 3 "~" H 10225 5850 50  0001 C CNN
 	1    10225 5650
@@
 F 0 "SW_CTL1.5u1" H 1125 4860 50  0000 C CNN
 F 1 "SW_Push" H 1125 4769 50  0000 C CNN
-F 2 "MX_Alps_Hybrid:MXOnly-1.25U-Hotswap" H 1125 4775 50  0001 C CNN
+F 2 "MX_Alps_Hybrid:MXOnly-1.25U-Hotswap-guide" H 1125 4775 50  0001 C CNN
 F 3 "~" H 1125 4775 50  0001 C CNN
 	1    1125 4575
@@
 F 0 "SW_ENT1.5u1" H 8275 4860 50  0000 C CNN
 F 1 "SW_Push" H 8275 4769 50  0000 C CNN
-F 2 "MX_Alps_Hybrid:MXOnly-1.5U-Hotswap" H 8275 4775 50  0001 C CNN
+F 2 "MX_Alps_Hybrid:MXOnly-1.5U-Hotswap-guide" H 8275 4775 50  0001 C CNN
 F 3 "~" H 8275 4775 50  0001 C CNN
 	1    8275 4575
@@
 F 0 "SW_RSFT1.75u1" H 8925 5935 50  0000 C CNN
 F 1 "SW_Push" H 8925 5844 50  0000 C CNN
-F 2 "MX_Alps_Hybrid:MXOnly-1.75U-Hotswap" H 8925 5850 50  0001 C CNN
+F 2 "MX_Alps_Hybrid:MXOnly-1.75U-Hotswap-guide" H 8925 5850 50  0001 C CNN
 F 3 "~" H 8925 5850 50  0001 C CNN
 	1    8925 5650
@@
 F 0 "SW_LSPC2u1" H 4375 7210 50  0000 C CNN
 F 1 "SW_Push" H 4375 7119 50  0000 C CNN
-F 2 "MX_Alps_Hybrid:MXOnly-2U-Hotswap-ReversedStabilizers" H 4375 7125 50  0001 C CNN
+F 2 "MX_Alps_Hybrid:MXOnly-2U-Hotswap-ReversedStabilizers-guide" H 4375 7125 50  0001 C CNN
 F 3 "~" H 4375 7125 50  0001 C CNN
 	1    4375 6925
@@
 F 0 "SW_LSPC2.25u1" H 4375 7360 50  0000 C CNN
 F 1 "SW_Push" H 4375 7269 50  0000 C CNN
-F 2 "MX_Alps_Hybrid:MXOnly-2.25U-Hotswap" H 4375 7275 50  0001 C CNN
+F 2 "MX_Alps_Hybrid:MXOnly-2.25U-Hotswap-guide" H 4375 7275 50  0001 C CNN
 F 3 "~" H 4375 7275 50  0001 C CNN
 	1    4375 7075
@@
 F 0 "SW_RCMD/HEN1.25u1" H 6975 7360 50  0000 C CNN
 F 1 "SW_Push" H 6975 7269 50  0000 C CNN
-F 2 "MX_Alps_Hybrid:MXOnly-1.25U-Hotswap" H 6975 7275 50  0001 C CNN
+F 2 "MX_Alps_Hybrid:MXOnly-1.25U-Hotswap-guide" H 6975 7275 50  0001 C CNN
 F 3 "~" H 6975 7275 50  0001 C CNN
 	1    6975 7075
@@
 F 0 "SW_RSPC6.25u1" H 5675 7360 50  0000 C CNN
 F 1 "SW_Push" H 5675 7269 50  0000 C CNN
-F 2 "MX_Alps_Hybrid:MXOnly-6.25U-Hotswap-ReversedStabilizers" H 5675 7275 50  0001 C CNN
+F 2 "MX_Alps_Hybrid:MXOnly-6.25U-Hotswap-ReversedStabilizers-guide" H 5675 7275 50  0001 C CNN
 F 3 "~" H 5675 7275 50  0001 C CNN
 	1    5675 7075
@@
 F 0 "SW_RSPC2u1" H 5675 7210 50  0000 C CNN
 F 1 "SW_Push" H 5675 7119 50  0000 C CNN
-F 2 "MX_Alps_Hybrid:MXOnly-2U-Hotswap-ReversedStabilizers" H 5675 7125 50  0001 C CNN
+F 2 "MX_Alps_Hybrid:MXOnly-2U-Hotswap-ReversedStabilizers-guide" H 5675 7125 50  0001 C CNN
 F 3 "~" H 5675 7125 50  0001 C CNN
 	1    5675 6925
@@
 F 0 "SW_MENU/ROPT1" H 8275 7360 50  0000 C CNN
 F 1 "SW_Push" H 8275 7269 50  0000 C CNN
-F 2 "MX_Alps_Hybrid:MXOnly-1U-Hotswap" H 8275 7275 50  0001 C CNN
+F 2 "MX_Alps_Hybrid:MXOnly-1U-Hotswap-guide" H 8275 7275 50  0001 C CNN
 F 3 "~" H 8275 7275 50  0001 C CNN
 	1    8275 7075
@@
 F 0 "SW_ROPT/KANA1.25u1" H 7625 7210 50  0000 C CNN
 F 1 "SW_Push" H 7625 7119 50  0000 C CNN
-F 2 "MX_Alps_Hybrid:MXOnly-1.25U-Hotswap" H 7625 7125 50  0001 C CNN
+F 2 "MX_Alps_Hybrid:MXOnly-1.25U-Hotswap-guide" H 7625 7125 50  0001 C CNN
 F 3 "~" H 7625 7125 50  0001 C CNN
 	1    7625 6925
@@
 F 0 "SW_CMD1.25u1" H 3075 7210 50  0000 C CNN
 F 1 "SW_Push" H 3075 7119 50  0000 C CNN
-F 2 "MX_Alps_Hybrid:MXOnly-1.25U-Hotswap" H 3075 7125 50  0001 C CNN
+F 2 "MX_Alps_Hybrid:MXOnly-1.25U-Hotswap-guide" H 3075 7125 50  0001 C CNN
 F 3 "~" H 3075 7125 50  0001 C CNN
 	1    3075 6925
@@
 F 0 "SW_MHEN/CMD1u1" H 3075 7360 50  0000 C CNN
 F 1 "SW_Push" H 3075 7269 50  0000 C CNN
-F 2 "MX_Alps_Hybrid:MXOnly-1U-Hotswap" H 3075 7275 50  0001 C CNN
+F 2 "MX_Alps_Hybrid:MXOnly-1U-Hotswap-guide" H 3075 7275 50  0001 C CNN
 F 3 "~" H 3075 7275 50  0001 C CNN
 	1    3075 7075
@@
 F 0 "SW_LSFT1.75u1" H 1125 5910 50  0000 C CNN
 F 1 "SW_Push" H 1125 5819 50  0000 C CNN
-F 2 "MX_Alps_Hybrid:MXOnly-1.75U-Hotswap" H 1125 5825 50  0001 C CNN
+F 2 "MX_Alps_Hybrid:MXOnly-1.75U-Hotswap-guide" H 1125 5825 50  0001 C CNN
 F 3 "~" H 1125 5825 50  0001 C CNN
 	1    1125 5625
@@
 F 0 "SW_BS1.5u1" H 8275 3610 50  0000 C CNN
 F 1 "SW_Push" H 8275 3519 50  0000 C CNN
-F 2 "MX_Alps_Hybrid:MXOnly-1.5U-Hotswap" H 8275 3525 50  0001 C CNN
+F 2 "MX_Alps_Hybrid:MXOnly-1.5U-Hotswap-guide" H 8275 3525 50  0001 C CNN
 F 3 "~" H 8275 3525 50  0001 C CNN
 	1    8275 3325
@@
 F 0 "SW_ROPT/KANA1.25u2" H 7625 7360 50  0000 C CNN
 F 1 "SW_Push" H 7625 7269 50  0000 C CNN
-F 2 "MX_Alps_Hybrid:MXOnly-1.25U-Hotswap" H 7625 7275 50  0001 C CNN
+F 2 "MX_Alps_Hybrid:MXOnly-1.25U-Hotswap-guide" H 7625 7275 50  0001 C CNN
 F 3 "~" H 7625 7275 50  0001 C CNN
 	1    7625 7075
@@
 F 0 "SW_CTL1.25u1" H 1125 4660 50  0000 C CNN
 F 1 "SW_Push" H 1125 4569 50  0000 C CNN
-F 2 "MX_Alps_Hybrid:MXOnly-1.5U-Hotswap" H 1125 4575 50  0001 C CNN
+F 2 "MX_Alps_Hybrid:MXOnly-1.5U-Hotswap-guide" H 1125 4575 50  0001 C CNN
 F 3 "~" H 1125 4575 50  0001 C CNN
 	1    1125 4375
@@
 F 0 "SW_CAPS1u1" H 1125 7360 50  0000 C CNN
 F 1 "SW_Push" H 1125 7269 50  0000 C CNN
-F 2 "MX_Alps_Hybrid:MXOnly-1U-Hotswap" H 1125 7275 50  0001 C CNN
+F 2 "MX_Alps_Hybrid:MXOnly-1U-Hotswap-guide" H 1125 7275 50  0001 C CNN
 F 3 "~" H 1125 7275 50  0001 C CNN
 	1    1125 7075
@@
 F 0 "SW_LongOPT1.25" H 1775 7360 50  0000 C CNN
 F 1 "SW_Push" H 1775 7269 50  0000 C CNN
-F 2 "MX_Alps_Hybrid:MXOnly-1.25U-Hotswap" H 1775 7275 50  0001 C CNN
+F 2 "MX_Alps_Hybrid:MXOnly-1.25U-Hotswap-guide" H 1775 7275 50  0001 C CNN
 F 3 "~" H 1775 7275 50  0001 C CNN
 	1    1775 7075
